Commit message: Nav2 added

File: src/pioneer_robot/resources/robots/pioneer.urdf (robot description, URDF)
Before this commit: robot pioneer3at_body, 18 links, 17 joints
Links:
- removed link laser_frame
- added link laser, mass 1e-5; collision box size=0.01 0.01 0.01; visual mesh filename=/home/winton/ros2_ws_part3/src/pioneer_robot/resources/mesh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
- link chassis: geometry collision mesh filename=/home/winton/ros2_ws_part3/src/pioneer_robot/resources/mesh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; visual mesh filename=/home/winton/ros2_ws_part3/src/pioneer_robot/resources/mesh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
- link p3at_back_left_axle: geometry collision box size=0.01 0.01 0.01; visual mesh filename=/home/winton/ros2_ws_part3/src/pioneer_robot/resources/mesh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
- link p3at_back_left_hub: geometry collision box size=0.01 0.01 0.01; visual mesh filename=/home/winton/ros2_ws_part3/src/pioneer_robot/resources/mesh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
- link p3at_back_left_wheel: geometry collision cylinder length=0.075 radius=0.111; visual mesh filename=/home/winton/ros2_ws_part3/src/pioneer_robot/resources/mesh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
- link p3at_back_right_axle: geometry collision box size=0.01 0.01 0.01; visual mesh filename=/home/winton/ros2_ws_part3/src/pioneer_robot/resources/mesh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
- link p3at_back_right_hub: geometry collision box size=0.01 0.01 0.01; visual mesh filename=/home/winton/ros2_ws_part3/src/pioneer_robot/resources/mesh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
- link p3at_back_right_wheel: geometry collision cylinder length=0.075 radius=0.111; visual mesh filename=/home/winton/ros2_ws_part3/src/pioneer_robot/resources/mesh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
- link p3at_front_left_axle: geometry collision box size=0.01 0.01 0.01; visual mesh filename=/home/winton/ros2_ws_part3/src/pioneer_robot/resources/mesh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
- link p3at_front_left_hub: geometry collision box size=0.01 0.01 0.01; visual mesh filename=/home/winton/ros2_ws_part3/src/pioneer_robot/resources/mesh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
- link p3at_front_left_wheel: geometry collision cylinder length=0.075 radius=0.111; visual mesh filename=/home/winton/ros2_ws_part3/src/pioneer_robot/resources/mesh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
- link p3at_front_right_axle: geometry collision box size=0.01 0.01 0.01; visual mesh filename=/home/winton/ros2_ws_part3/src/pioneer_robot/resources/mesh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
- link p3at_front_right_hub: geometry collision box size=0.01 0.01 0.01; visual mesh filename=/home/winton/ros2_ws_part3/src/pioneer_robot/resources/mesh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
- link p3at_front_right_wheel: geometry collision cylinder length=0.075 radius=0.111; visual mesh filename=/home/winton/ros2_ws_part3/src/pioneer_robot/resources/mesh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
- link top_plate: geometry collision box size=0.1 0.1 0.1; visual mesh filename=/home/winton/ros2_ws_part3/src/pioneer_robot/resources/mesh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
Joints:
- joint laser_joint: child laser_frame -> laser
